File: 00_simple/00_led/led/led.sch (KiCad schematic (older format))
At the start: 3 parts

Commit message: add annotation
Parts:
- gave numbers to parts that had none: 3
Changed lines of the file:
@@
 $EndDescr
 $Comp
-L Device:LED D?
+L Device:LED D1
 U 1 1 5B87612A
 P 5150 4300
-F 0 "D?" V 5188 4183 50  0000 R CNN
+F 0 "D1" V 5188 4183 50  0000 R CNN
 F 1 "OSR5JA3Z74A" V 5097 4183 50  0000 R CNN
 F 2 "" H 5150 4300 50  0001 C CNN
@@
 $EndComp
 $Comp
-L Device:R R?
+L Device:R R1
 U 1 1 5B8761AC
 P 5150 3450
-F 0 "R?" H 5220 3496 50  0000 L CNN
+F 0 "R1" H 5220 3496 50  0000 L CNN
 F 1 "640" H 5220 3405 50  0000 L CNN
 F 2 "" V 5080 3450 50  0001 C CNN
@@
 	5150 4450 5150 4950
 $Comp
-L power:GND #PWR?
+L power:GND #PWR01
 U 1 1 5B876387
 P 5150 4950
-F 0 "#PWR?" H 5150 4700 50  0001 C CNN
+F 0 "#PWR01" H 5150 4700 50  0001 C CNN
 F 1 "GND" H 5155 4777 50  0000 C CNN
 F 2 "" H 5150 4950 50  0001 C CNN
@@
 $EndComp
 $Comp
-L Switch:SW_SPST SW?
+L Switch:SW_SPST SW1
 U 1 1 5B8766D2
 P 5950 3050
-F 0 "SW?" H 5950 3285 50  0000 C CNN
+F 0 "SW1" H 5950 3285 50  0000 C CNN
 F 1 "SW_SPST" H 5950 3194 50  0000 C CNN
 F 2 "" H 5950 3050 50  0001 C CNN

Commit message: add ERC
Connections:
- net labels added: For_ERC
- wire segments 5 -> 6
Changed lines of the file:
@@
 Wire Wire Line
 	5150 3050 5150 3300
+$Comp
+L power:PWR_FLAG #FLG0101
+U 1 1 5B8774C0
+P 7200 4650
+F 0 "#FLG0101" H 7200 4725 50  0001 C CNN
+F 1 "PWR_FLAG" H 7200 4824 50  0000 C CNN
+F 2 "" H 7200 4650 50  0001 C CNN
+F 3 "~" H 7200 4650 50  0001 C CNN
+	1    7200 4650
+	1    0    0    -1
+$EndComp
+$Comp
+L power:GND #PWR0101
+U 1 1 5B877517
+P 7200 4950
+F 0 "#PWR0101" H 7200 4700 50  0001 C CNN
+F 1 "GND" H 7205 4777 50  0000 C CNN
+F 2 "" H 7200 4950 50  0001 C CNN
+F 3 "" H 7200 4950 50  0001 C CNN
+	1    7200 4950
+	1    0    0    -1
+$EndComp
+Wire Wire Line
+	7200 4650 7200 4950
+$Comp
+L power:PWR_FLAG #FLG0102
+U 1 1 5B877573
+P 6750 3050
+F 0 "#FLG0102" H 6750 3125 50  0001 C CNN
+F 1 "PWR_FLAG" H 6750 3224 50  0000 C CNN
+F 2 "" H 6750 3050 50  0001 C CNN
+F 3 "~" H 6750 3050 50  0001 C CNN
+	1    6750 3050
+	1    0    0    -1
+$EndComp
+Wire Notes Line
+	6850 5250 7550 5250
+Wire Notes Line
+	7550 5250 7550 4150
+Wire Notes Line
+	7550 4150 6850 4150
+Wire Notes Line
+	6850 4150 6850 5250
+Text Label 6900 4250 0    50   ~ 0
+For_ERC
 $EndSCHEMATC
