File: 00_simple/00_led/led/led.sch (KiCad schematic (older format))
At the start: 3 parts, among them SW1 SW_SPST

Commit message: assign footprints
Parts:
- D1: footprint (none) -> LED_THT:LED_D3.0mm
- R1: footprint (none) -> Resistor_THT:R_Axial_DIN0207_L6.3mm_D2.5mm_P7.62mm_Horizontal
- SW1: footprint (none) -> mylib:TVGP01-G73BB
Changed lines of the file:
@@
 F 0 "D1" V 5188 4183 50  0000 R CNN
 F 1 "OSR5JA3Z74A" V 5097 4183 50  0000 R CNN
-F 2 "" H 5150 4300 50  0001 C CNN
+F 2 "LED_THT:LED_D3.0mm" H 5150 4300 50  0001 C CNN
 F 3 "~" H 5150 4300 50  0001 C CNN
 	1    5150 4300
@@
 F 0 "R1" H 5220 3496 50  0000 L CNN
 F 1 "640" H 5220 3405 50  0000 L CNN
-F 2 "" V 5080 3450 50  0001 C CNN
+F 2 "Resistor_THT:R_Axial_DIN0207_L6.3mm_D2.5mm_P7.62mm_Horizontal" V 5080 3450 50  0001 C CNN
 F 3 "~" H 5150 3450 50  0001 C CNN
 	1    5150 3450
@@
 F 0 "SW1" H 5950 3285 50  0000 C CNN
 F 1 "SW_SPST" H 5950 3194 50  0000 C CNN
-F 2 "" H 5950 3050 50  0001 C CNN
+F 2 "mylib:TVGP01-G73BB" H 5950 3050 50  0001 C CNN
 F 3 "" H 5950 3050 50  0001 C CNN
 	1    5950 3050
