File: 00_simple/01_inverting_operational_amplifier/Untitled.sch (KiCad schematic (older format))
At the start: 3 parts, among them U1 OPAMP

Commit message: change circuit
Parts:
- added R3, R4: 1k, symbol Device:R
- R1, R2: value R -> 10k
Connections:
- net labels added: 5V
- wire segments 17 -> 21
Changed lines of the file:
@@
 EESchema Schematic File Version 4
+LIBS:Untitled-cache
 EELAYER 26 0
 EELAYER END
@@
 F 3 "" H 5300 3200 50  0001 C CNN
 	1    5300 3200
-	1    0    0    1
-$EndComp
-$Comp
-L Device:R R1
-U 1 1 5B97D420
-P 4150 3100
-F 0 "R1" H 4220 3146 50  0000 L CNN
-F 1 "R" H 4220 3055 50  0000 L CNN
-F 2 "" V 4080 3100 50  0001 C CNN
-F 3 "~" H 4150 3100 50  0001 C CNN
-	1    4150 3100
-	0    -1   -1   0
-$EndComp
-$Comp
-L Device:R R2
-U 1 1 5B97D48B
-P 4750 2500
-F 0 "R2" H 4820 2546 50  0000 L CNN
-F 1 "R" H 4820 2455 50  0000 L CNN
-F 2 "" V 4680 2500 50  0001 C CNN
-F 3 "~" H 4750 2500 50  0001 C CNN
-	1    4750 2500
-	0    -1   -1   0
+	1    0    0    -1
 $EndComp
 $Comp
 L power:GND #PWR01
 U 1 1 5B97DB6C
-P 4450 3900
-F 0 "#PWR01" H 4450 3650 50  0001 C CNN
-F 1 "GND" H 4455 3727 50  0000 C CNN
-F 2 "" H 4450 3900 50  0001 C CNN
-F 3 "" H 4450 3900 50  0001 C CNN
-	1    4450 3900
-	1    0    0    -1
-$EndComp
-$Comp
-L power:GND #PWR02
-U 1 1 5B97DB9E
-P 5500 2800
-F 0 "#PWR02" H 5500 2550 50  0001 C CNN
-F 1 "GND" H 5505 2627 50  0000 C CNN
-F 2 "" H 5500 2800 50  0001 C CNN
-F 3 "" H 5500 2800 50  0001 C CNN
-	1    5500 2800
-	1    0    0    -1
-$EndComp
-$Comp
-L power:PWR_FLAG #FLG02
-U 1 1 5B97DBD7
-P 5500 3850
-F 0 "#FLG02" H 5500 3925 50  0001 C CNN
-F 1 "PWR_FLAG" H 5500 4024 50  0000 C CNN
-F 2 "" H 5500 3850 50  0001 C CNN
-F 3 "~" H 5500 3850 50  0001 C CNN
-	1    5500 3850
+P 5200 4600
+F 0 "#PWR01" H 5200 4350 50  0001 C CNN
+F 1 "GND" H 5205 4427 50  0000 C CNN
+F 2 "" H 5200 4600 50  0001 C CNN
+F 3 "" H 5200 4600 50  0001 C CNN
+	1    5200 4600
 	1    0    0    -1
 $EndComp
@@
 L power:PWR_FLAG #FLG01
 U 1 1 5B97DC09
-P 3400 3100
-F 0 "#FLG01" H 3400 3175 50  0001 C CNN
-F 1 "PWR_FLAG" H 3400 3274 50  0000 C CNN
-F 2 "" H 3400 3100 50  0001 C CNN
-F 3 "~" H 3400 3100 50  0001 C CNN
-	1    3400 3100
+P 6600 3200
+F 0 "#FLG01" H 6600 3275 50  0001 C CNN
+F 1 "PWR_FLAG" H 6600 3374 50  0000 C CNN
+F 2 "" H 6600 3200 50  0001 C CNN
+F 3 "~" H 6600 3200 50  0001 C CNN
+	1    6600 3200
 	1    0    0    -1
 $EndComp
@@
 L power:PWR_FLAG #FLG03
 U 1 1 5B97DC3B
-P 6400 3200
-F 0 "#FLG03" H 6400 3275 50  0001 C CNN
-F 1 "PWR_FLAG" H 6400 3374 50  0000 C CNN
-F 2 "" H 6400 3200 50  0001 C CNN
-F 3 "~" H 6400 3200 50  0001 C CNN
-	1    6400 3200
+P 2600 2200
+F 0 "#FLG03" H 2600 2275 50  0001 C CNN
+F 1 "PWR_FLAG" H 2600 2374 50  0000 C CNN
+F 2 "" H 2600 2200 50  0001 C CNN
+F 3 "~" H 2600 2200 50  0001 C CNN
+	1    2600 2200
 	1    0    0    -1
 $EndComp
-Text Label 6100 3150 0    50   ~ 0
+Text Label 6550 3350 0    50   ~ 0
 Vo
-Text Label 3650 3050 0    50   ~ 0
-Vi
-Text Label 4650 2650 0    50   ~ 0
+Text Label 5450 3950 0    50   ~ 0
 I2->
 Text Label 4800 3400 0    50   ~ 0
 Vp
-Text Label 4100 3250 0    50   ~ 0
+Text Label 4050 3600 0    50   ~ 0
 I1->
-Wire Wire Line
-	4450 3300 4450 3900
-Wire Wire Line
-	5000 3300 4450 3300
-Wire Wire Line
-	3400 3100 4000 3100
-Wire Wire Line
-	4600 2500 4450 2500
-Wire Wire Line
-	5850 3200 6400 3200
-Wire Wire Line
-	5850 2500 4900 2500
-Wire Wire Line
-	5850 3200 5850 2500
-Connection ~ 5850 3200
-Wire Wire Line
-	5600 3200 5850 3200
-Wire Wire Line
-	4450 3100 5000 3100
-Wire Wire Line
-	4450 2500 4450 3100
-Connection ~ 4450 3100
-Wire Wire Line
-	4300 3100 4450 3100
 Text Label 4800 3050 0    50   ~ 0
 Vn
+$Comp
+L Device:R R2
+U 1 1 5B991214
+P 5550 3800
+F 0 "R2" V 5343 3800 50  0000 C CNN
+F 1 "10k" V 5434 3800 50  0000 C CNN
+F 2 "" V 5480 3800 50  0001 C CNN
+F 3 "~" H 5550 3800 50  0001 C CNN
+	1    5550 3800
+	0    1    1    0
+$EndComp
+$Comp
+L Device:R R1
+U 1 1 5B99129F
+P 4150 3300
+F 0 "R1" V 4300 3300 50  0000 C CNN
+F 1 "10k" V 4034 3300 50  0000 C CNN
+F 2 "" V 4080 3300 50  0001 C CNN
+F 3 "~" H 4150 3300 50  0001 C CNN
+	1    4150 3300
+	0    1    1    0
+$EndComp
 Wire Wire Line
-	5200 2900 5200 2650
+	4700 3800 4700 3300
+Connection ~ 4700 3300
 Wire Wire Line
-	5200 2650 5500 2650
+	4700 3300 5000 3300
 Wire Wire Line
-	5500 2650 5500 2800
+	5700 3800 6000 3800
 Wire Wire Line
-	5500 3850 5500 3950
+	6000 3800 6000 3200
 Wire Wire Line
-	5500 3950 5200 3950
+	6000 3200 5600 3200
+Connection ~ 5200 4400
+$Comp
+L Device:R R4
+U 1 1 5B992333
+P 2900 3650
+F 0 "R4" H 2970 3696 50  0000 L CNN
+F 1 "1k" H 2970 3605 50  0000 L CNN
+F 2 "" V 2830 3650 50  0001 C CNN
+F 3 "~" H 2900 3650 50  0001 C CNN
+	1    2900 3650
+	1    0    0    -1
+$EndComp
+$Comp
+L Device:R R3
+U 1 1 5B992DE8
+P 2900 2650
+F 0 "R3" H 2970 2696 50  0000 L CNN
+F 1 "1k" H 2970 2605 50  0000 L CNN
+F 2 "" V 2830 2650 50  0001 C CNN
+F 3 "~" H 2900 2650 50  0001 C CNN
+	1    2900 2650
+	1    0    0    -1
+$EndComp
 Wire Wire Line
-	5200 3950 5200 3500
+	2900 3100 2900 2800
+Wire Wire Line
+	2900 3100 2900 3500
+Connection ~ 2900 3100
+Wire Wire Line
+	2600 2200 2900 2200
+Wire Wire Line
+	5200 2200 5200 2900
+Connection ~ 2900 2200
+Wire Wire Line
+	2900 2200 2900 2500
+$Comp
+L power:PWR_FLAG #FLG02
+U 1 1 5B9949BF
+P 3500 3300
+F 0 "#FLG02" H 3500 3375 50  0001 C CNN
+F 1 "PWR_FLAG" H 3500 3200 50  0000 C CNN
+F 2 "" H 3500 3300 50  0001 C CNN
+F 3 "~" H 3500 3300 50  0001 C CNN
+	1    3500 3300
+	1    0    0    -1
+$EndComp
+Wire Wire Line
+	5200 4400 5200 4600
+Text Label 3500 3550 0    50   ~ 0
+Vi
+Wire Wire Line
+	2900 4400 5200 4400
+Wire Wire Line
+	4300 3300 4700 3300
+Wire Wire Line
+	3500 3300 4000 3300
+Wire Wire Line
+	2900 3100 5000 3100
+Wire Wire Line
+	2900 2200 5200 2200
+Wire Wire Line
+	6000 3200 6600 3200
+Connection ~ 6000 3200
+Wire Wire Line
+	5200 4400 6600 4400
+Wire Wire Line
+	4700 3800 5400 3800
+Wire Wire Line
+	5200 3500 5200 4400
+Wire Wire Line
+	2900 3800 2900 4400
+Text Label 2550 2350 0    50   ~ 0
+5V
 $EndSCHEMATC
