File: 00_simple/03_npn_transistor/Untitled.sch (KiCad schematic (older format))
At the start: 4 parts, among them Q1 2SC1815

Commit message: update 03
Parts:
- D1: value LED -> OSR5JA3Z74A
- Q1: value 2SC1815 -> 2SC1815GR
- R1: value R -> 10k
- R2: value R -> 100
Changed lines of the file:
@@
 EESchema Schematic File Version 4
+LIBS:Untitled-cache
 EELAYER 26 0
 EELAYER END
@@
 P 5600 3800
 F 0 "Q1" H 5791 3846 50  0000 L CNN
-F 1 "2SC1815" H 5791 3755 50  0000 L CNN
+F 1 "2SC1815GR" H 5791 3755 50  0000 L CNN
 F 2 "" H 5800 3900 50  0001 C CNN
 F 3 "~" H 5600 3800 50  0001 C CNN
@@
 P 5700 2250
 F 0 "D1" V 5738 2133 50  0000 R CNN
-F 1 "LED" V 5647 2133 50  0000 R CNN
+F 1 "OSR5JA3Z74A" V 5647 2133 50  0000 R CNN
 F 2 "" H 5700 2250 50  0001 C CNN
 F 3 "~" H 5700 2250 50  0001 C CNN
@@
 P 5700 2950
 F 0 "R2" H 5770 2996 50  0000 L CNN
-F 1 "R" H 5770 2905 50  0000 L CNN
+F 1 "100" H 5770 2905 50  0000 L CNN
 F 2 "" V 5630 2950 50  0001 C CNN
 F 3 "~" H 5700 2950 50  0001 C CNN
@@
 P 4950 3800
 F 0 "R1" V 4743 3800 50  0000 C CNN
-F 1 "R" V 4834 3800 50  0000 C CNN
+F 1 "10k" V 4834 3800 50  0000 C CNN
 F 2 "" V 4880 3800 50  0001 C CNN
 F 3 "~" H 4950 3800 50  0001 C CNN
