File: 00_simple/04_pnp_transistor/Untitled.sch (KiCad schematic (older format))
At the start: 4 parts, among them Q1 2SA1015

Commit message: update 04
Parts:
- D1: value LED -> OSR5JA3Z74A
- Q1: value 2SA1015 -> 2SA1015GR
- R1: value R -> 10k
- R2: value R -> 100
Changed lines of the file:
@@
 P 5500 3500
 F 0 "Q1" H 5691 3546 50  0000 L CNN
-F 1 "2SA1015" H 5691 3455 50  0000 L CNN
+F 1 "2SA1015GR" H 5691 3455 50  0000 L CNN
 F 2 "" H 5700 3600 50  0001 C CNN
 F 3 "~" H 5500 3500 50  0001 C CNN
@@
 P 5600 4200
 F 0 "R2" H 5670 4246 50  0000 L CNN
-F 1 "R" H 5670 4155 50  0000 L CNN
+F 1 "100" H 5670 4155 50  0000 L CNN
 F 2 "" V 5530 4200 50  0001 C CNN
 F 3 "~" H 5600 4200 50  0001 C CNN
@@
 P 4800 3500
 F 0 "R1" V 4593 3500 50  0000 C CNN
-F 1 "R" V 4684 3500 50  0000 C CNN
+F 1 "10k" V 4684 3500 50  0000 C CNN
 F 2 "" V 4730 3500 50  0001 C CNN
 F 3 "~" H 4800 3500 50  0001 C CNN
@@
 P 5600 4800
 F 0 "D1" V 5638 4683 50  0000 R CNN
-F 1 "LED" V 5547 4683 50  0000 R CNN
+F 1 "OSR5JA3Z74A" V 5547 4683 50  0000 R CNN
 F 2 "" H 5600 4800 50  0001 C CNN
 F 3 "~" H 5600 4800 50  0001 C CNN
