File: 00_simple/05_nmos_fet/Untitled.sch (KiCad schematic (older format))
At the start: 5 parts, among them Q1 Q_NMOS_GDS

Commit message: update 05
Parts:
- D1: value LED -> OSR5JA3Z74A
- R3: value R -> 100
Changed lines of the file:
@@
 EESchema Schematic File Version 4
+LIBS:Untitled-cache
 EELAYER 26 0
 EELAYER END
@@
 P 5500 2550
 F 0 "R3" H 5570 2596 50  0000 L CNN
-F 1 "R" H 5570 2505 50  0000 L CNN
+F 1 "100" H 5570 2505 50  0000 L CNN
 F 2 "" V 5430 2550 50  0001 C CNN
 F 3 "~" H 5500 2550 50  0001 C CNN
@@
 P 5500 2000
 F 0 "D1" V 5538 1883 50  0000 R CNN
-F 1 "LED" V 5447 1883 50  0000 R CNN
+F 1 "OSR5JA3Z74A" V 5447 1883 50  0000 R CNN
 F 2 "" H 5500 2000 50  0001 C CNN
 F 3 "~" H 5500 2000 50  0001 C CNN
